Commit message: feat: add camera_optical link and joint

File: src/sitl_launcher/urdf/iris_depth.urdf.xacro (robot description, xacro)
@@ -55,3 +55,9 @@
     <origin xyz="0.135 0 0" rpy="0 -0.26 0"/>
   </joint>
+<link name="camera_optical_link"/>
+<joint name="camera_optical_joint" type="fixed">
+  <parent link="camera_link"/>
+  <child link="camera_optical_link"/>
+  <origin xyz="0 0 0" rpy="0 0.26 0"/>
+</joint>
 </robot>
